File: PCB/LED_Snowboard_V4/io.kicad_sch (KiCad schematic)
At the start: 59 parts, among them J1 Conn_01x04, J10 XT60PW-F, J12 Power Switch, J2 Conn_01x04, J3 Conn_01x04, J4 XT60PW-M, J5 XT60PW-M, J7 LED Data, J8 Sensor Input, J9 Encoder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

Commit message: makerfaire
Parts:
- added C17, C18: .1uF, Capacitor_SMD:C_0603_1608Metric_Pad1.08x0.95mm_HandSolder, symbol Device:C
- added D13: D_Schottky, Package_TO_SOT_SMD:TO-263-3_TabPin2, symbol Device:D_Schottky
- added D14, D15: D_Zener, Diode_SMD:D_SOD-123, symbol Device:D_Zener
- added F2, F4: Fuse, Fuse:Fuse_0603_1608Metric_Pad1.05x0.95mm_HandSolder, symbol Device:Fuse
- added Q3, Q4: X0202NN, Package_TO_SOT_SMD:TO-252-2, symbol Triac_Thyristor:X0202NN
- added R22, R23: 1k, Resistor_SMD:R_0603_1608Metric_Pad0.98x0.95mm_HandSolder, symbol Device:R
- C1, C10, C11, C2, C3, C4, C5, C6, C7, C8, C9: footprint (none) -> Capacitor_SMD:C_0603_1608Metric_Pad1.08x0.95mm_HandSolder
- D3, D4, D5: footprint (none) -> Diode_SMD:D_SOD-123
- F1: footprint (none) -> SF-3812F3500T-2:SF-3812F3500T-2
- H1, H2: footprint (none) -> MountingHole:MountingHole_4.3mm_M4_Pad
- J1: value Conn_01x04 -> Charge_Balance; footprint (none) -> Connector_JST:JST_XA_B04B-XASK-1_1x04_P2.50mm_Vertical
- J10: value XT60PW-F -> Output
- J12, J7, J8: footprint (none) -> Connector_JST:JST_XA_B03B-XASK-1_1x03_P2.50mm_Vertical
- J2: value Conn_01x04 -> Bat2_Balance; footprint (none) -> Connector_JST:JST_XA_S04B-XASK-1N-BN_1x04_P2.50mm_Horizontal
- J3: value Conn_01x04 -> Bat1_Balance; footprint (none) -> Connector_JST:JST_XA_S04B-XASK-1N-BN_1x04_P2.50mm_Horizontal
- J4: value XT60PW-M -> Bat1
- J5: value XT60PW-M -> Bat2
- J9: footprint (none) -> Connector_JST:JST_XA_B05B-XASK-1_1x05_P2.50mm_Vertical
- L1, L2: footprint (none) -> SnapEDA Library:IND_SRR4818A-150M
- Q1, Q2: footprint (none) -> Package_DFN_QFN:PQFN-8-EP_6x5mm_P1.27mm_Generic
- R1, R11, R12, R13, R14, R15, R16, R17, R18, R19, R2, R20, R21, R3, R4, R5, R6, R7, R8, R9: footprint (none) -> Resistor_SMD:R_0603_1608Metric_Pad0.98x0.95mm_HandSolder
- R10: footprint (none) -> SnapEDA Library:RES_WSK12161L000FEA
Connections:
- net +3V3: now also D15.1 (K), F2.2, Q4.2 (A), Q4.4 (A); no longer C7.2, C9.2, L2.2, U5.1 (FB)
- net +5V: now also D14.1 (K), F4.2, Q3.2 (A), Q3.4 (A); no longer C6.2, C8.2, L1.2, U4.1 (FB)
- net GND: now also J1.4 (Pin_4), J2.4 (Pin_4), J3.4 (Pin_4), C17.1, C18.1, D13.3 (A), Q3.1 (K), Q4.1 (K), R22.2, R23.2; no longer J1.1 (Pin_1), J2.1 (Pin_1), J3.1 (Pin_1)
- net VCC: now also R10.3; no longer R10.2
- net at J1.3 (Pin_3), J2.3 (Pin_3), J3.3 (Pin_3): now also R4.1, R5.1; no longer R2.1, R3.2
- net at F1.2, U2.10 (VIN+), U2.8 (VBUS): now also R10.2, D13.2 (K); no longer R10.1
- net at J1.2 (Pin_2), J2.2 (Pin_2), J3.2 (Pin_2): now also R2.1, R3.2; no longer R4.1, R5.1
- new net: C17.2, D14.2 (A), Q3.3 (G), R22.1
- new net: C6.2, C8.2, F4.1, L1.2, U4.1 (FB)
- new net: C7.2, C9.2, F2.1, L2.2, U5.1 (FB)
- new net: C18.2, D15.2 (A), Q4.3 (G), R23.1
- new net: J1.1 (Pin_1), J2.1 (Pin_1), J3.1 (Pin_1), R1.1
Other:
- moved on the sheet: C10, C11, C2, C3, C4, C5, C6, C7, C8, C9, J12, L1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

Commit message: Added Ram
Added Ram. need to finish DRC checks
Parts:
- added J6: ~, Connector_AMASS:AMASS_XT30U-M_1x02_P5.0mm_Vertical, symbol Dustins_Symbols:xt30
- J12: footprint Connector_JST:JST_XA_B03B-XASK-1_1x03_P2.50mm_Vertical -> Connector_Molex:Molex_Nano-Fit_105309-xx03_1x03_P2.50mm_Vertical
Connections:
- net +BATT: now also J6.2
- net GND: now also J6.1
Changed lines of the file:
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@@
   (junction (at 175.26 40.64) (diameter 0) (color 0 0 0 0)
   )
+  (junction (at 45.72 58.42) (diameter 0) (color 0 0 0 0)
+  )
   (junction (at 124.46 35.56) (diameter 0) (color 0 0 0 0)
   )
@@
   )
   (junction (at 199.39 74.93) (diameter 0) (color 0 0 0 0)
+  )
+  (junction (at 43.18 78.74) (diameter 0) (color 0 0 0 0)
   )
   (junction (at 194.31 45.72) (diameter 0) (color 0 0 0 0)
@@
     (stroke (width 0) (type default))
   )
+  (wire (pts (xy 39.37 76.2) (xy 45.72 76.2))
+    (stroke (width 0) (type default))
+  )
   (wire (pts (xy 63.5 158.75) (xy 63.5 176.53))
     (stroke (width 0) (type default))
@@
     (stroke (width 0) (type default))
   )
+  (wire (pts (xy 39.37 78.74) (xy 43.18 78.74))
+    (stroke (width 0) (type default))
+  )
   (wire (pts (xy 93.98 81.28) (xy 97.79 81.28))
     (stroke (width 0) (type default))
@@
     (stroke (width 0) (type default))
   )
-  (wire (pts (xy 43.18 64.77) (xy 43.18 60.96))
+  (wire (pts (xy 43.18 82.55) (xy 43.18 78.74))
     (stroke (width 0) (type default))
   )
@@
     (stroke (width 0) (type default))
   )
+  (wire (pts (xy 45.72 76.2) (xy 45.72 58.42))
+    (stroke (width 0) (type default))
+  )
   (wire (pts (xy 36.83 168.91) (xy 45.72 168.91))
+    (stroke (width 0) (type default))
+  )
+  (wire (pts (xy 43.18 78.74) (xy 43.18 60.96))
     (stroke (width 0) (type default))
   )
@@
       (effects (font (size 1.27 1.27)) hide)
     )
+    (pin "2")
     (pin "3")
-    (pin "2")
     (instances
       (project "LED_Snowboard_V4"
@@
     )
   )
-  (symbol (lib_id "power:GND") (at 43.18 64.77 0) (unit 1)
+  (symbol (lib_id "power:GND") (at 43.18 82.55 0) (unit 1)
     (in_bom yes) (on_board yes) (dnp no) (fields_autoplaced)
-    (property "Reference" "#PWR011" (at 43.18 71.12 0)
-      (effects (font (size 1.27 1.27)) hide)
-    )
-    (property "Value" "GND" (at 43.18 69.85 0)
-      (effects (font (size 1.27 1.27)))
-    )
-    (property "Footprint" "" (at 43.18 64.77 0)
-      (effects (font (size 1.27 1.27)) hide)
-    )
-    (property "Datasheet" "" (at 43.18 64.77 0)
+    (property "Reference" "#PWR011" (at 43.18 88.9 0)
+      (effects (font (size 1.27 1.27)) hide)
+    )
+    (property "Value" "GND" (at 43.18 87.63 0)
+      (effects (font (size 1.27 1.27)))
+    )
+    (property "Footprint" "" (at 43.18 82.55 0)
+      (effects (font (size 1.27 1.27)) hide)
+    )
+    (property "Datasheet" "" (at 43.18 82.55 0)
       (effects (font (size 1.27 1.27)) hide)
     )
@@
       (effects (font (size 1.27 1.27)) (justify right))
     )
-    (property "Footprint" "Connector_JST:JST_XA_B03B-XASK-1_1x03_P2.50mm_Vertical" (at 129.54 20.32 0)
+    (property "Footprint" "Connector_Molex:Molex_Nano-Fit_105309-xx03_1x03_P2.50mm_Vertical" (at 129.54 20.32 0)
       (effects (font (size 1.27 1.27)) hide)
     )
@@
         )
       )
+    )
+  )
+  (symbol (lib_id "Dustins_Symbols:xt30") (at 26.67 73.66 0) (unit 1)
+    (in_bom yes) (on_board yes) (dnp no) (fields_autoplaced)
+    (property "Reference" "J6" (at 30.48 71.12 0)
+      (effects (font (size 1.27 1.27)))
+    )
+    (property "Value" "~" (at 26.67 73.66 0)
+      (effects (font (size 1.27 1.27)))
+    )
+    (property "Footprint" "Connector_AMASS:AMASS_XT30U-M_1x02_P5.0mm_Vertical" (at 26.67 73.66 0)
+      (effects (font (size 1.27 1.27)) hide)
+    )
+    (property "Datasheet" "" (at 26.67 73.66 0)
+      (effects (font (size 1.27 1.27)) hide)
+    )
+    (pin "1")
+    (pin "2")
+    (instances
+      (project "LED_Snowboard_V4"
+        (path "/69eedaaa-0c0b-424a-87de-b98a25a250e0/609d0ec3-3d5e-48f8-8437-e8dde642f153"
+          (reference "J6") (unit 1)
+        )
+      )

Commit message: Finished PCB with all feedback
Parts:
- C10, C11: value C -> .1uF
- L1: value 4.7uF -> 4.7uH
- L2: value 3.9uF -> 3.9uH
Changed lines of the file:
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@@
       (effects (font (size 1.27 1.27)))
     )
-    (property "Value" "C" (at 236.22 16.51 90)
+    (property "Value" ".1uF" (at 237.49 16.51 90)
       (effects (font (size 1.27 1.27)))
     )
@@
       (effects (font (size 1.27 1.27)))
     )
-    (property "Value" "3.9uF" (at 165.1 73.66 90)
+    (property "Value" "3.9uH" (at 165.1 73.66 90)
       (effects (font (size 1.27 1.27)))
     )
@@
       (effects (font (size 1.27 1.27)))
     )
-    (property "Value" "C" (at 210.82 16.51 90)
+    (property "Value" ".1uF" (at 209.55 16.51 90)
       (effects (font (size 1.27 1.27)))
     )
@@
       (effects (font (size 1.27 1.27)))
     )
-    (property "Value" "4.7uF" (at 165.1 34.29 90)
-      (effects (font (size 1.27 1.27)))
-    )
+    (property "Value" "4.7uH" (at 165.1 34.29 90)
+      (effects (font (size 1.27 1.27)))
+    )

Commit message: updated control pcb
updated to add high side switching as well as added voltage divider and adjusted layout
Parts:
- removed D1, D2: SD05_SOD323, Diode_SMD:D_SOD-323, symbol Diode:SD05_SOD323
- removed D14, D15: D_Zener, Diode_SMD:D_SOD-123, symbol Device:D_Zener
- removed D3, D4, D5: D_Schottky, Diode_SMD:D_SOD-123, symbol Device:D_Schottky
- removed F2, F4: Fuse, Fuse:Fuse_0603_1608Metric_Pad1.05x0.95mm_HandSolder, symbol Device:Fuse
- removed Q3, Q4: X0202NN, Package_TO_SOT_SMD:TO-252-2, symbol Triac_Thyristor:X0202NN
- removed R23: 1k, Resistor_SMD:R_0603_1608Metric_Pad0.98x0.95mm_HandSolder, symbol Device:R
- added C19, C20: .1uF, Capacitor_SMD:C_0603_1608Metric_Pad1.08x0.95mm_HandSolder, symbol Device:C
- added U10: 1EDL8011XUMA1, PG-DSO-8-92_INF, symbol 2025-06-29_03-38-02:1EDL8011XUMA1
- C17: value .1uF -> 10uF
- C18: value .1uF -> 10n
- F1: value Fuse -> 35A Fuse
- Q1, Q2: value ~ -> IRFH5300TRPBF
- R15: value 10k -> 422k
- R16: value 1k -> 100
- R17: value 1k -> 500k
- R22: value 1k -> 100k
Connections:
- net +3V3: now also C7.2, C9.2, L2.2, U5.1 (FB)
- net +5V: now also C6.2, C8.2, L1.2, U4.1 (FB)
- net GATE_SIGNAL: now also U10.2 (IN); no longer R15.1, R16.1, R17.1
- net GND: now also J10.1, C19.1, C20.1, U10.1 (GND); no longer C18.1, Q1.1 (S), Q2.1 (S)
- net VCC: now also C17.2, Q1.3 (D), Q2.3 (D), R17.2, U10.8 (VIN); no longer J10.2
- net at U6.11 (B3): now also R21.2
- net at U6.12 (B2): now also R20.2
- net at U6.13 (B1): now also R19.2
- net BAT: now reaches R22.1
- net BAT: now also R17.1, C20.2; no longer C17.2
- net at Q1.2 (G): now also Q2.2 (G), C19.2, U10.6 (GATE); no longer R16.2
- net at C18.2: now also R16.2
- new net: J10.2, Q1.1 (S), Q2.1 (S), U10.7 (VS)
- new net: R15.1, U10.5 (ILIMIT)
- new net: R16.1, U10.4 (CFP)
- new net: C18.1, U10.3 (CFN)
Other:
- note added: "0.1% resistors should be used"
- note added: "Cell Monitor Parasitic Draw (Worst Case) Cell 1 draw - 28uA Cell 2 Draw - 56uA Cell 3 Draw - 84uA"
- note added: "Current limit set to 40.6A"
- note added: "Gain = 6 Fc = ~19.1Hz Current Draw (Worst Case) = 21uA"
- note added: "High side switching is required to avoid issues with 12V on LED Data lines"
- note added: "I=12k/(Rds*R)"
- note added: "Theoretical max current for V2 2280 leds is 32.8A"
- note added: "shunt power = 1.06W @ 32.8A"
- moved on the sheet: C6, C7, C8, C9, Q1, R10, R14, R19, R20, R21
